Commit message: inclusao da camera no moveit

File: denso_robot_moveit_config/robots/vs050/srdf/denso_robot_macro.srdf.xacro (robot description, xacro)
@@ -5,5 +5,5 @@
     A URDF file must exist for this robot as well, where the joints and the links that are referenced are defined
 -->
-  <xacro:macro name="denso_robot_srdf" params="namespace">
+  <xacro:macro name="denso_robot_srdf" params="namespace basic_camera:=false">
     <!--GROUPS - Representation of a set of joints and links. This can be useful for specifying DOF to plan for, defining arms, end effectors, etc-->
     <!--LINKS - When a link is specified, the parent joint of that link (if it exists) is automatically included-->
@@ -32,4 +32,8 @@
 	<disable_collisions link1="${namespace}J3" link2="${namespace}J5" reason="Never"/>
 	<disable_collisions link1="${namespace}J4" link2="${namespace}J5" reason="Adjacent"/>
+    <!-- Touch tool with RealSense D405: only the mounting pair is excluded -->
+    <xacro:if value="${basic_camera}">
+      <disable_collisions link1="${namespace}J6" link2="${namespace}toucher_link" reason="Adjacent"/>
+    </xacro:if>
   </xacro:macro>
 </robot>

File: denso_robot_moveit_config/srdf/denso_robot.srdf.xacro (robot description, xacro)
@@ -5,5 +5,6 @@
   <!-- parameters -->
   <xacro:arg name="namespace" default="" />
+  <xacro:arg name="basic_camera" default="false" />
   <xacro:include filename="$(find denso_robot_moveit_config)/robots/$(arg model)/srdf/denso_robot_macro.srdf.xacro"/>
-  <xacro:denso_robot_srdf namespace="$(arg namespace)"/>
+  <xacro:denso_robot_srdf namespace="$(arg namespace)" basic_camera="$(arg basic_camera)"/>
 </robot>
